File: schematics/gpa/gpa.kicad_sch (KiCad schematic)
At the start: 17 parts, among them U1 HC-SR04, U2 HC-SR04

Commit message: update
Small update, waiting hardware
Parts:
- removed A1: Arduino_Nano_v3.x, Module:Arduino_Nano, symbol MCU_Module:Arduino_Nano_v3.x
- removed LF1, LF2, LF3, LS1, LS2, LS3: LED, symbol Device:LED
- removed R7: 0, symbol Device:R
- removed RSW1: KSK-1A66-2030, KSK-1A66-2030:SW_KSK-1A66-2030, symbol KSK-1A66-2030:KSK-1A66-2030
- added A1: A000067, Arduino Mega 2560 Rev3:ARDUINO_A000067, symbol Arduino Mega 2560 Rev3:A000067
- added D1, D2, D3, D4: LED, Connector_PinHeader_2.54mm:PinHeader_1x02_P2.54mm_Vertical, symbol Device:LED
- added L1: LCD-16X2, Display:LCD-016N002L, symbol LCD 16x2:LCD-16X2
- added RSW1: SW_Reed, Connector_PinHeader_2.54mm:PinHeader_1x02_P2.54mm_Vertical, symbol Switch:SW_Reed
- added SW1, SW2, SW3, SW4: SW_Push, Connector_PinHeader_2.54mm:PinHeader_1x02_P2.54mm_Vertical, symbol Switch:SW_Push
- R1: value 10K -> 330Ω; footprint (none) -> Resistor_THT:R_Axial_DIN0207_L6.3mm_D2.5mm_P7.62mm_Horizontal
- R2, R3, R4, R5, R6: value 0 -> 10K; footprint (none) -> Resistor_THT:R_Axial_DIN0207_L6.3mm_D2.5mm_P7.62mm_Horizontal
Connections:
- net at U1.1 (VCC), U2.1 (VCC): now also A1.5V_2 (+5V_2), RSW1.1, SW1.1, SW2.1, SW3.1, SW4.1
- net at U1.2 (TRIG): now also A1.17
- net at U1.3 (ECHO): now also A1.16
- net at R3.2: now also R2.2, R4.2, R5.2, R6.2, U1.4 (GND), U2.4 (GND), A1.GND4, D1.2 (A), D2.2 (A), D3.2 (A), D4.2 (A)
- net at U2.2 (TRIG): now also A1.15
- net at U2.3 (ECHO): now also A1.14
- net at R1.2: now also A1.GND1, L1.2 (VDD)
- new net: L1.16 (K), R1.1
- new net: A1.5V_1 (+5V_1), L1.1 (VSS)
- new net: A1.34, L1.10 (DB3)
- new net: A1.36, L1.11 (DB4)
- new net: A1.38, L1.12 (DB5)
- new net: A1.40, L1.13 (DB6)
- new net: A1.42, L1.14 (DB7)
- new net: A1.3, L1.15 (A)
- new net: A1.2, L1.3 (VO)
- new net: A1.22, L1.4 (RS)
- new net: A1.24, L1.5 (R/W)
- new net: A1.26, L1.6 (E)
- new net: A1.28, L1.7 (DB0)
- new net: A1.30, L1.8 (DB1)
- new net: A1.32, L1.9 (DB2)
- new net: A1.44, R6.1, SW1.2
- new net: A1.5, D2.1 (K)
- new net: A1.50, R3.1, SW4.2
- new net: A1.52, R2.1, RSW1.2
- new net: A1.46, R5.1, SW2.2
- new net: A1.4, D1.1 (K)
- new net: A1.48, R4.1, SW3.2
- new net: A1.6, D3.1 (K)
- new net: A1.7, D4.1 (K)
Other:
- company: Andrew G Hill -> Andrew Hill
